Commit message: Lab 2Step 3

File: Step2/table.urdf.xacro (robot description, xacro)
@@ -3,4 +3,5 @@
   <!-- Xacro files here -->
   <xacro:include filename="table_macro.xacro" />
+  <xacro:include filename="materials.xacro" />
   <!-- Create the frame -->
   <link name="world" />

File: Step2/table_macro.xacro (robot description, xacro)
@@ -1,4 +1,4 @@
-<?xml vexrsion="1.0"?>
-<robot xmlns:xacro="https://wiki.ros.org/xacro">
+<?xml version="1.0"?>
+<robot xmlns:xacro="http://www.ros.org/wiki/xacro">
   <!-- Table Parameters given in the question -->
   <xacro:macro name="table" params="prefix parent *origin">
@@ -20,4 +20,5 @@
     <link name="${prefix}top">
       <visual>
+        <!-- top frame is centered on the TOP surface -->
         <origin xyz="0 0 ${-table_thickness/2}" rpy="0 0 0"/>
         <geometry>
@@ -28,10 +29,11 @@
     </link>
     <!-- Tangent to the sides -->
-    <xacro: value="${table_length/2 - leg_radius}" />
-    <xacro: value="${table_width/2 - leg_radius}" />
+    <xacro:property name="x_off" value="${table_length/2 - leg_radius}" />
+    <xacro:property name="y_off" value="${table_width/2 - leg_radius}" />
     <!-- Leg macro -->
     <xacro:macro name="leg" params="name x y">
       <link name="${prefix}${name}">
         <visual>
+          <!-- leg frame is at TOP of leg -->
           <origin xyz="0 0 ${-leg_length/2}" rpy="0 0 0"/>
           <geometry>
@@ -44,11 +46,13 @@
         <parent link="${prefix}top"/>
         <child link="${prefix}${name}"/>
+        <!-- put leg TOP at underside of tabletop -->
+        <origin xyz="${x} ${y} ${-table_thickness}" rpy="0 0 0"/>
       </joint>
     </xacro:macro>
-    <!-- Four legs -->
-    <xacro:leg name="leg1" />
-    <xacro:leg name="leg2" />
-    <xacro:leg name="leg3" />
-    <xacro:leg name="leg4" />
+    <!-- Four legs: tangent to sides and fully under top -->
+    <xacro:leg name="leg1" x="${ x_off}"  y="${ y_off}"/>
+    <xacro:leg name="leg2" x="${ x_off}"  y="${-y_off}"/>
+    <xacro:leg name="leg3" x="${-x_off}"  y="${ y_off}"/>
+    <xacro:leg name="leg4" x="${-x_off}"  y="${-y_off}"/>
   </xacro:macro>
 </robot>
